Commit message: repaired

File: src/dossarm_description/urdf/dossarm.urdf.xacro (robot description, xacro)
@@ -1,658 +1,376 @@
 <?xml version="1.0" ?>
-<!-- =================================================================================== -->
-<!-- |    This document was autogenerated by xacro from /home/nils/Documents/Studium/Studienarbeit/DossArm/src/dossarm_description/urdf/dossarm.urdf.xacro | -->
-<!-- |    EDITING THIS FILE BY HAND IS NOT RECOMMENDED                                 | -->
-<!-- =================================================================================== -->
-<robot name="moveo_description">
-    <!-- https://bitbucket.org/theconstructcore/my-robotic-manipulator/src/master/urdf/links_joints.xacro -->
-    <link name="world" />
-    <!-- <xacro:include filename="$(find dossarm_description)/urdf/links_joints.xacro" /> -->
-    <link name="base">
-<inertial>
-            <mass value="0.1" />
-            <origin rpy="1.5707 0 0" xyz="0  0 0" />
-            <inertia ixx="0.03" ixy="0.0" ixz="0.0" iyy="0.03" iyz="0.0" izz="0.03" />
-        </inertial>
-        <collision>
-            <origin rpy="1.5707 0 0" xyz="0  0 0" />
-            <geometry>
-                <mesh filename="package://dossarm_description/meshes/Motor_1_Case.stl" scale="0.00 0.001 0.001" />
-            </geometry>
-        </collision>
-        <visual>
-            <origin rpy="1.5707 0 0" xyz="0  0 0" />
-            <geometry>
-                <mesh filename="package://dossarm_description/meshes/Motor_1_Case.stl" scale="0.001 0.001 0.001" />
-            </geometry>
-            <material name="">
-                <color rgba="0.79216 0.81961 0.93333 1" />
-            </material>
-        </visual>
+<robot name="moveo_description" xmlns:xacro="http://www.ros.org/wiki/xacro">
+     <xacro:include filename="$(find dossarm_description)/urdf/links_joints.xacro" />
+    <xacro:property name="path_to_meshes" value="package://dossarm_description/meshes" />
+    <xacro:m_link_mesh name="base"
+        origin_xyz="0 0 0"
+        origin_rpy="1.5707 0 0"
+        meshfile_visual= "package://dossarm_description/meshes/Motor_1_Case.stl"
+        meshfile_collision= "package://dossarm_description/meshes/Motor_1_Case.stl"
+        mass="0.1"
+        ixx="0.03"
+        ixy="0.0"
+        ixz="0.0"
+        iyy= "0.03"
+        iyz= "0.0"
+        izz="0.03"
+    />
+    <!-- dummy link -->
+    <link name="world">
     </link>
-    <joint name="world_to_base=" type="fixed">
+    <joint name="odom_joint" type="fixed">
+        <origin xyz="0 0 -1" rpy="0 0 0" />
         <parent link="world" />
         <child link="base" />
-        <origin rpy="0 0 0" xyz="0  0 -1" />
     </joint>
-    <link name="Motor_1">
-<inertial>
-            <mass value="0.1" />
-            <origin rpy="1.5708 0 0" xyz="0 0 0" />
-            <inertia ixx="0.03" ixy="0.0" ixz="0.0" iyy="0.03" iyz="0.0" izz="0.03" />
-        </inertial>
-        <collision>
-            <origin rpy="1.5708 0 0" xyz="0 0 0" />
-            <geometry>
-                <mesh filename="package://dossarm_description/meshes/PH54_200.stl" scale="0.00 0.001 0.001" />
-            </geometry>
-        </collision>
-        <visual>
-            <origin rpy="1.5708 0 0" xyz="0 0 0" />
-            <geometry>
-                <mesh filename="package://dossarm_description/meshes/PH54_200.stl" scale="0.001 0.001 0.001" />
-            </geometry>
-            <material name="">
-                <color rgba="0.79216 0.81961 0.93333 1" />
-            </material>
-        </visual>
-    </link>
-    <joint name="joint_base-motor_1" type="fixed">
-        <axis xyz="0 0 0" />
-        <limit effort="5" lower="-1.5707" upper="1.5707" velocity="1" />
-        <origin rpy="0 0 0" xyz="0 0 0.064" />
-        <parent link="base" />
-        <child link="Motor_1" />
-    </joint>
-    <transmission name="trans_joint_base-motor_1">
-        <type>hardware_interface/PositionJointInterface</type>
-        <joint name="joint_base-motor_1">
-            <hardwareInterface>hardware_interface/PositionJointInterface</hardwareInterface>
-        </joint>
-        <actuator name="motor_joint_base-motor_1">
-            <hardwareInterface>hardware_interface/PositionJointInterface</hardwareInterface>
-            <mechanicalReduction>1</mechanicalReduction>
-        </actuator>
-    </transmission>
-    <link name="Link_1">
-<inertial>
-            <mass value="0.1" />
-            <origin rpy="1.5708 0 0" xyz="0 0  0" />
-            <inertia ixx="0.03" ixy="0.0" ixz="0.0" iyy="0.03" iyz="0.0" izz="0.03" />
-        </inertial>
-        <collision>
-            <origin rpy="1.5708 0 0" xyz="0 0  0" />
-            <geometry>
-                <mesh filename="package://dossarm_description/meshes/Motor_2_Case.stl" scale="0.00 0.001 0.001" />
-            </geometry>
-        </collision>
-        <visual>
-            <origin rpy="1.5708 0 0" xyz="0 0  0" />
-            <geometry>
-                <mesh filename="package://dossarm_description/meshes/Motor_2_Case.stl" scale="0.001 0.001 0.001" />
-            </geometry>
-            <material name="">
-                <color rgba="0.79216 0.81961 0.93333 1" />
-            </material>
-        </visual>
-    </link>
-    <joint name="Joint_1" type="continuous">
-        <axis xyz="0 0 1" />
-        <limit effort="5" lower="-1.5707" upper="1.5707" velocity="1" />
-        <origin rpy="0 0 0" xyz="0 0 0.095" />
-        <parent link="Motor_1" />
-        <child link="Link_1" />
-    </joint>
-    <transmission name="trans_Joint_1">
-        <type>hardware_interface/PositionJointInterface</type>
-        <joint name="Joint_1">
-            <hardwareInterface>hardware_interface/PositionJointInterface</hardwareInterface>
-        </joint>
-        <actuator name="motor_Joint_1">
-            <hardwareInterface>hardware_interface/PositionJointInterface</hardwareInterface>
-            <mechanicalReduction>1</mechanicalReduction>
-        </actuator>
-    </transmission>
-    <link name="Motor_2">
-<inertial>
-            <mass value="0.1" />
-            <origin rpy="0 0 0" xyz=" 0 0 0" />
-            <inertia ixx="0.03" ixy="0.0" ixz="0.0" iyy="0.03" iyz="0.0" izz="0.03" />
-        </inertial>
-        <collision>
-            <origin rpy="0 0 0" xyz=" 0 0 0" />
-            <geometry>
-                <mesh filename="package://dossarm_description/meshes/PH54_200_Bearings.stl" scale="0.00 0.001 0.001" />
-            </geometry>
-        </collision>
-        <visual>
-            <origin rpy="0 0 0" xyz=" 0 0 0" />
-            <geometry>
-                <mesh filename="package://dossarm_description/meshes/PH54_200_Bearings.stl" scale="0.001 0.001 0.001" />
-            </geometry>
-            <material name="">
-                <color rgba="0.79216 0.81961 0.93333 1" />
-            </material>
-        </visual>
-    </link>
-    <joint name="joint_Link_2-motor_1" type="fixed">
-        <axis xyz="0 0 0" />
-        <limit effort="5" lower="-1.5707" upper="1.5707" velocity="1" />
-        <origin rpy="0 0 1.5708" xyz="-0.00575 0 0  " />
-        <parent link="Link_1" />
-        <child link="Motor_2" />
-    </joint>
-    <transmission name="trans_joint_Link_2-motor_1">
-        <type>hardware_interface/PositionJointInterface</type>
-        <joint name="joint_Link_2-motor_1">
-            <hardwareInterface>hardware_interface/PositionJointInterface</hardwareInterface>
-        </joint>
-        <actuator name="motor_joint_Link_2-motor_1">
-            <hardwareInterface>hardware_interface/PositionJointInterface</hardwareInterface>
-            <mechanicalReduction>1</mechanicalReduction>
-        </actuator>
-    </transmission>
-    <link name="shoulder">
-<inertial>
-            <mass value="0.1" />
-            <origin rpy="0 0 0" xyz="0 0 0" />
-            <inertia ixx="0.03" ixy="0.0" ixz="0.0" iyy="0.03" iyz="0.0" izz="0.03" />
-        </inertial>
-        <collision>
-            <origin rpy="0 0 0" xyz="0 0 0" />
-            <geometry>
-                <mesh filename="package://dossarm_description/meshes/Shoulder_complete.stl" scale="0.00 0.001 0.001" />
-            </geometry>
-        </collision>
-        <visual>
-            <origin rpy="0 0 0" xyz="0 0 0" />
-            <geometry>
-                <mesh filename="package://dossarm_description/meshes/Shoulder_complete.stl" scale="0.001 0.001 0.001" />
-            </geometry>
-            <material name="">
-                <color rgba="0.79216 0.81961 0.93333 1" />
-            </material>
-        </visual>
-    </link>
-    <joint name="Joint_2" type="revolute">
-        <axis xyz="1 0 0" />
-        <limit effort="5" lower="-1.5707" upper="1.5707" velocity="1" />
-        <origin rpy="0 0 1.5708" xyz="0 -0.00575 0" />
-        <parent link="Motor_2" />
-        <child link="shoulder" />
-    </joint>
-    <transmission name="trans_Joint_2">
-        <type>hardware_interface/PositionJointInterface</type>
-        <joint name="Joint_2">
-            <hardwareInterface>hardware_interface/PositionJointInterface</hardwareInterface>
-        </joint>
-        <actuator name="motor_Joint_2">
-            <hardwareInterface>hardware_interface/PositionJointInterface</hardwareInterface>
-            <mechanicalReduction>1</mechanicalReduction>
-        </actuator>
-    </transmission>
-    <link name="Motor_3">
-<inertial>
-            <mass value="0.1" />
-            <origin rpy="0 0 0 " xyz=" 0 0 0" />
-            <inertia ixx="0.03" ixy="0.0" ixz="0.0" iyy="0.03" iyz="0.0" izz="0.03" />
-        </inertial>
-        <collision>
-            <origin rpy="0 0 0 " xyz=" 0 0 0" />
-            <geometry>
-                <mesh filename="package://dossarm_description/meshes/PH54_200_Bearings.stl" scale="0.00 0.001 0.001" />
-            </geometry>
-        </collision>
-        <visual>
-            <origin rpy="0 0 0 " xyz=" 0 0 0" />
-            <geometry>
-                <mesh filename="package://dossarm_description/meshes/PH54_200_Bearings.stl" scale="0.001 0.001 0.001" />
-            </geometry>
-            <material name="">
-                <color rgba="0.79216 0.81961 0.93333 1" />
-            </material>
-        </visual>
-    </link>
-    <joint name="UpperArm_Motor_3_Connection" type="fixed">
-        <axis xyz="0 0 0" />
-        <limit effort="5" lower="-1.5707" upper="1.5707" velocity="1" />
-        <origin rpy="0 0  0" xyz="0 0.00575 0.1" />
-        <parent link="shoulder" />
-        <child link="Motor_3" />
-    </joint>
-    <transmission name="trans_UpperArm_Motor_3_Connection">
-        <type>hardware_interface/PositionJointInterface</type>
-        <joint name="UpperArm_Motor_3_Connection">
-            <hardwareInterface>hardware_interface/PositionJointInterface</hardwareInterface>
-        </joint>
-        <actuator name="motor_UpperArm_Motor_3_Connection">
-            <hardwareInterface>hardware_interface/PositionJointInterface</hardwareInterface>
-            <mechanicalReduction>1</mechanicalReduction>
-        </actuator>
-    </transmission>
-    <link name="upperarm">
-<inertial>
-            <mass value="0.1" />
-            <origin rpy="0 0 0 " xyz="0 0 0" />
-            <inertia ixx="0.03" ixy="0.0" ixz="0.0" iyy="0.03" iyz="0.0" izz="0.03" />
-        </inertial>
-        <collision>
-            <origin rpy="0 0 0 " xyz="0 0 0" />
-            <geometry>
-                <mesh filename="package://dossarm_description/meshes/upperarm_complete.stl" scale="0.00 0.001 0.001" />
-            </geometry>
-        </collision>
-        <visual>
-            <origin rpy="0 0 0 " xyz="0 0 0" />
-            <geometry>
-                <mesh filename="package://dossarm_description/meshes/upperarm_complete.stl" scale="0.001 0.001 0.001" />
-            </geometry>
-            <material name="">
-                <color rgba="0.79216 0.81961 0.93333 1" />
-            </material>
-        </visual>
-    </link>
-    <joint name="Joint_3" type="revolute">
-        <axis xyz="1 0 0" />
-        <limit effort="5" lower="-1.5707" upper="1.5707" velocity="1" />
-        <origin rpy="0 0 1.5708" xyz="0 -0.00575 0" />
-        <parent link="Motor_3" />
-        <child link="upperarm" />
-    </joint>
-    <transmission name="trans_Joint_3">
-        <type>hardware_interface/PositionJointInterface</type>
-        <joint name="Joint_3">
-            <hardwareInterface>hardware_interface/PositionJointInterface</hardwareInterface>
-        </joint>
-        <actuator name="motor_Joint_3">
-            <hardwareInterface>hardware_interface/PositionJointInterface</hardwareInterface>
-            <mechanicalReduction>1</mechanicalReduction>
-        </actuator>
-    </transmission>
-    <link name="Motor_4">
-<inertial>
-            <mass value="0.1" />
-            <origin rpy="0 0 0" xyz="0 0 0" />
-            <inertia ixx="0.03" ixy="0.0" ixz="0.0" iyy="0.03" iyz="0.0" izz="0.03" />
-        </inertial>
-        <collision>
-            <origin rpy="0 0 0" xyz="0 0 0" />
-            <geometry>
-                <mesh filename="package://dossarm_description/meshes/PH54_200_Bearings.stl" scale="0.00 0.001 0.001" />
-            </geometry>
-        </collision>
-        <visual>
-            <origin rpy="0 0 0" xyz="0 0 0" />
-            <geometry>
-                <mesh filename="package://dossarm_description/meshes/PH54_200_Bearings.stl" scale="0.001 0.001 0.001" />
-            </geometry>
-            <material name="">
-                <color rgba="0.79216 0.81961 0.93333 1" />
-            </material>
-        </visual>
-    </link>
-    <joint name="motor4_forearm_connection" type="fixed">
-        <axis xyz="0 0 0" />
-        <limit effort="5" lower="-1.5707" upper="1.5707" velocity="1" />
-        <origin rpy="0 0 1.5708" xyz=" -0.00575 0 0.343041 " />
-        <parent link="upperarm" />
-        <child link="Motor_4" />
-    </joint>
-    <transmission name="trans_motor4_forearm_connection">
-        <type>hardware_interface/PositionJointInterface</type>
-        <joint name="motor4_forearm_connection">
-            <hardwareInterface>hardware_interface/PositionJointInterface</hardwareInterface>
-        </joint>
-        <actuator name="motor_motor4_forearm_connection">
-            <hardwareInterface>hardware_interface/PositionJointInterface</hardwareInterface>
-            <mechanicalReduction>1</mechanicalReduction>
-        </actuator>
-    </transmission>
-    <link name="forearm_upper">
-<inertial>
-            <mass value="0.1" />
-            <origin rpy="0 0 0" xyz="0 0 0" />
-            <inertia ixx="0.03" ixy="0.0" ixz="0.0" iyy="0.03" iyz="0.0" izz="0.03" />
-        </inertial>
-        <collision>
-            <origin rpy="0 0 0" xyz="0 0 0" />
-            <geometry>
-                <mesh filename="package://dossarm_description/meshes/forearm_upper_complete.stl" scale="0.00 0.001 0.001" />
-            </geometry>
-        </collision>
-        <visual>
-            <origin rpy="0 0 0" xyz="0 0 0" />
-            <geometry>
-                <mesh filename="package://dossarm_description/meshes/forearm_upper_complete.stl" scale="0.001 0.001 0.001" />
-            </geometry>
-            <material name="">
-                <color rgba="0.79216 0.81961 0.93333 1" />
-            </material>
-        </visual>
-    </link>
-    <joint name="Joint_4" type="revolute">
-        <axis xyz="1 0 0" />
-        <limit effort="5" lower="-1.5707" upper="1.5707" velocity="1" />
-        <origin rpy="0 0  1.5708 " xyz=" 0   -0.00575  0" />
-        <parent link="Motor_4" />
-        <child link="forearm_upper" />
-    </joint>
-    <transmission name="trans_Joint_4">
-        <type>hardware_interface/PositionJointInterface</type>
-        <joint name="Joint_4">
-            <hardwareInterface>hardware_interface/PositionJointInterface</hardwareInterface>
-        </joint>
-        <actuator name="motor_Joint_4">
-            <hardwareInterface>hardware_interface/PositionJointInterface</hardwareInterface>
-            <mechanicalReduction>1</mechanicalReduction>
-        </actuator>
-    </transmission>
-    <link name="Motor_5">
-<inertial>
-            <mass value="0.1" />
-            <origin rpy="0 0 0" xyz="0 0 0" />
-            <inertia ixx="0.03" ixy="0.0" ixz="0.0" iyy="0.03" iyz="0.0" izz="0.03" />
-        </inertial>
-        <collision>
-            <origin rpy="0 0 0" xyz="0 0 0" />
-            <geometry>
-                <mesh filename="package://dossarm_description/meshes/H54P-100_M54P-040.stl" scale="0.00 0.001 0.001" />
-            </geometry>
-        </collision>
-        <visual>
-            <origin rpy="0 0 0" xyz="0 0 0" />
-            <geometry>
-                <mesh filename="package://dossarm_description/meshes/H54P-100_M54P-040.stl" scale="0.001 0.001 0.001" />
-            </geometry>
-            <material name="">
-                <color rgba="0.79216 0.81961 0.93333 1" />
-            </material>
-        </visual>
-    </link>
-    <joint name="forearm_lower_Motor5_connection" type="fixed">
-        <axis xyz="0 0 0" />
-        <limit effort="5" lower="-1.5707" upper="1.5707" velocity="1" />
-        <origin rpy="1.5708 0 0" xyz=" 0 0 0.1775  " />
-        <parent link="forearm_upper" />
-        <child link="Motor_5" />
-    </joint>
-    <transmission name="trans_forearm_lower_Motor5_connection">
-        <type>hardware_interface/PositionJointInterface</type>
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