Commit message: Bugfix axis_xyz all zeroes --> NAN Quaterion error

File: src/dossarm_description/urdf/dossarm.urdf.xacro (robot description, xacro)
@@ -1,11 +1,18 @@
 <?xml version="1.0" ?>
-<robot name="moveo_description" xmlns:xacro="http://www.ros.org/wiki/xacro">
-     <xacro:include filename="$(find dossarm_description)/urdf/links_joints.xacro" />
+<robot name="dossarm_description" xmlns:xacro="http://www.ros.org/wiki/xacro">
+    <xacro:include filename="$(find dossarm_description)/urdf/links_joints.xacro" />
     <xacro:property name="path_to_meshes" value="package://dossarm_description/meshes" />
-    <xacro:m_link_mesh name="base"
+     <link name="world">
+    </link>
+      <joint name="odom_joint" type="fixed">
+        <origin xyz="0 0 -1" rpy="0 0 0" />
+        <parent link="world" />
+        <child link="base_link" />
+    </joint>
+    <xacro:m_link_mesh name="base_link"
         origin_xyz="0 0 0"
         origin_rpy="1.5707 0 0"
-        meshfile_visual= "package://dossarm_description/meshes/Motor_1_Case.stl"
-        meshfile_collision= "package://dossarm_description/meshes/Motor_1_Case.stl"
+        meshfile_visual= "${path_to_meshes}/Motor_1_Case.stl"
+        meshfile_collision= "${path_to_meshes}/Motor_1_Case.stl"
         mass="0.1"
         ixx="0.03"
@@ -16,12 +23,4 @@
         izz="0.03"
     />
-    <!-- dummy link -->
-    <link name="world">
-    </link>
-    <joint name="odom_joint" type="fixed">
-        <origin xyz="0 0 -1" rpy="0 0 0" />
-        <parent link="world" />
-        <child link="base" />
-    </joint>
      <xacro:m_link_mesh name="Motor_1"
     origin_xyz="0 0 0"
@@ -37,15 +36,9 @@
     izz="0.03"
     />
-     <xacro:m_joint name= "dummyjoint_base_to_motor_1"
-        type="fixed"
+     <xacro:m_joint_fixed name= "dummyjoint_base_to_motor_1"
         origin_xyz= "0 0 0.064"
         origin_rpy="0 0 0"
-        axis_xyz="0 0 0"
-        parent="base"
+        parent="base_link"
         child="Motor_1"
-        limit_l="-1.5707"
-        limit_u="1.5707"
-        limit_v="1"
-        limit_e="5"
     />
     <xacro:m_link_mesh name="Link_1"
@@ -87,15 +80,9 @@
     izz="0.03"
     />
-          <xacro:m_joint name= "dummyjoint_Link_1_to_Motor_1"
-        type="fixed"
+          <xacro:m_joint_fixed name= "dummyjoint_Link_1_to_Motor_1"
         origin_xyz= "-0.00575 0 0"
         origin_rpy="0 0 1.5708"
-        axis_xyz="0 0 0"
         parent="Link_1"
         child="Motor_2"
-        limit_l="-1.5707"
-        limit_u="1.5707"
-        limit_v="1"
-        limit_e="5"
     />
    <xacro:m_link_mesh name="shoulder"
@@ -112,9 +99,9 @@
     izz="0.03"
     />
-       <xacro:m_joint name= "Joint_2"
+    <xacro:m_joint name= "Joint_2"
         type="revolute"
         origin_xyz= "0 -0.00575 0"
         origin_rpy="0 0 1.5708"
-        axis_xyz="0 0 0"
+        axis_xyz="1 0 0"
         parent="Motor_2"
         child="shoulder"
@@ -137,15 +124,9 @@
     izz="0.03"
     />
-       <xacro:m_joint name= "dummyJoint_Motor_3_to_UpperArm"
-        type="fixed"
+       <xacro:m_joint_fixed name= "dummyJoint_Motor_3_to_UpperArm"
         origin_xyz= "0 0.00575 0.1"
         origin_rpy="0 0 0"
-        axis_xyz="0 0 0"
         parent="shoulder"
         child="Motor_3"
-        limit_l="-1.5707"
-        limit_u="1.5707"
-        limit_v="1"
-        limit_e="5"
     />
     <xacro:m_link_mesh name="upperarm"
@@ -187,15 +168,9 @@
     izz="0.03"
     />
-        <xacro:m_joint name= "dummyJoint_Motor_4_to_forearm"
-        type="fixed"
+        <xacro:m_joint_fixed name= "dummyJoint_Motor_4_to_forearm"
         origin_xyz= "-0.00575 0 0.343041 "
         origin_rpy="0 0 1.5708"
-        axis_xyz="0 0 0"
         parent="upperarm"
         child="Motor_4"
-        limit_l="-1.5707"
-        limit_u="1.5707"
-        limit_v="1"
-        limit_e="5"
     />
     <xacro:m_link_mesh name="forearm_upper"
@@ -237,15 +212,9 @@
     izz="0.03"
     />
-     <xacro:m_joint name= "dummyJoint_forearm_upper_to_Motor_5"
-        type="fixed"
+     <xacro:m_joint_fixed name= "dummyJoint_forearm_upper_to_Motor_5"
         origin_xyz= "0  0  0.1775"
         origin_rpy="1.5708 0 0 "
-        axis_xyz="0 0 0"
         parent="forearm_upper"
         child="Motor_5"
-        limit_l="-1.5707"
-        limit_u="1.5707"
-        limit_v="1"
-        limit_e="5"
     />
 <xacro:m_link_mesh name="forearm_lower"
@@ -287,15 +256,9 @@
     izz="0.03"
     />
- <xacro:m_joint name= "dummyJoint_Motor_6_Wrist_Connection"
-        type="fixed"
+ <xacro:m_joint_fixed name= "dummyJoint_Motor_6_Wrist_Connection"
         origin_xyz= "0.039 0 0.124233"
         origin_rpy="0 1.5708  0 "
-        axis_xyz="0 0 0"
         parent="forearm_lower"
         child="Motor_6"
-        limit_l="-1.5707"
-        limit_u="1.5707"
-        limit_v="1"
-        limit_e="5"
     />
      <xacro:m_link_mesh name="wrist"
@@ -337,15 +300,9 @@
         izz="0.03"
     />
- <xacro:m_joint name= "dummyJoint_Wrist_to_Motor_7"
-        type="fixed"
+ <xacro:m_joint_fixed name= "dummyJoint_Wrist_to_Motor_7"
         origin_xyz= "0.039 0 0.082"
         origin_rpy= "1.5708 0 1.5708"
-        axis_xyz="0 1 0"
         parent="wrist"
         child="Motor_7"
-        limit_l="-1.5707"
-        limit_u="1.5707"
-        limit_v="1"
-        limit_e="5"
     />
    <xacro:m_link_mesh name="arm_ph42"
@@ -374,3 +331,6 @@
         limit_e="5"
     />
+     <gazebo>
+        <plugin name="gazebo_ros_control" filename="libgazebo_ros_control.so"/>
+    </gazebo>
 </robot>

File: src/dossarm_description/urdf/links_joints.xacro (robot description, xacro)
@@ -2,5 +2,5 @@
 <robot xmlns:xacro="http://www.ros.org/wiki/xacro">
 <!-- https://bitbucket.org/theconstructcore/my-robotic-manipulator/src/master/urdf/links_joints.xacro -->
-  <xacro:macro name="m_joint" params="name type axis_xyz origin_rpy origin_xyz parent child  limit_e limit_l limit_u limit_v mimic_joint:='' mimic_multiplier:=1 mimic_offset:=0 ">
+  <xacro:macro name="m_joint" params="name type axis_xyz origin_rpy origin_xyz parent child limit_e limit_l limit_u limit_v mimic_joint:='' mimic_multiplier:=1 mimic_offset:=0 ">
     <joint name="${name}" type="${type}">
       <axis xyz="${axis_xyz}" />
@@ -9,5 +9,4 @@
       <parent link="${parent}" />
       <child link="${child}" />
-      <!-- <calibration rising = "${calibration}"/> -->
       <xacro:if value ="${mimic_joint !=''}">
       <mimic joint="${mimic_joint}" multiplier="${mimic_multiplier}" offset="${mimic_offset}" />
@@ -15,14 +14,21 @@
     </joint>
     <transmission name="trans_${name}">
-      <type>hardware_interface/PositionJointInterface</type>
+      <type>transmission_interface/SimpleTransmission</type>
       <joint name="${name}">
-        <hardwareInterface>hardware_interface/PositionJointInterface</hardwareInterface>
+        <hardwareInterface>hardware_interface/EffortJointInterface</hardwareInterface>
       </joint>
       <actuator name="motor_${name}">
-        <hardwareInterface>hardware_interface/PositionJointInterface</hardwareInterface>
+        <hardwareInterface>hardware_interface/EffortJointInterface</hardwareInterface>
         <mechanicalReduction>1</mechanicalReduction>
       </actuator>
     </transmission>
   </xacro:macro>
+<xacro:macro name="m_joint_fixed" params="name origin_rpy origin_xyz parent child ">
+    <joint name="${name}" type="fixed">
+      <origin rpy="${origin_rpy}" xyz="${origin_xyz}" />
+      <parent link="${parent}" />
+      <child link="${child}" />
+    </joint>
+</xacro:macro>
   <xacro:macro name="m_link_mesh" params="name origin_xyz origin_rpy meshfile_visual meshfile_collision mass ixx ixy ixz iyy iyz izz">
     <link name="${name}">
@@ -35,5 +41,5 @@
         <origin rpy="${origin_rpy}" xyz="${origin_xyz}" />
         <geometry>
-          <mesh filename="${meshfile_collision}" scale="0.00 0.001 0.001"/>
+          <mesh filename="${meshfile_collision}" scale="0.001 0.001 0.001"/>/>
         </geometry>
       </collision>
@@ -49,4 +55,5 @@
     </link>
   </xacro:macro>
+<!--
 <xacro:macro name="m_link_cylinder" params="name origin_xyz origin_rpy radius length mass ixx ixy ixz iyy iyz izz">
     <link name="${name}">
@@ -90,4 +97,4 @@
       </visual>
     </link>
-  </xacro:macro>
+  </xacro:macro> -->
 </robot>

Commit message: added Moveit Gazebo support

File: src/dossarm_description/urdf/dossarm.urdf.xacro (robot description, xacro)
@@ -5,6 +5,6 @@
      <link name="world">
     </link>
-      <joint name="odom_joint" type="fixed">
-        <origin xyz="0 0 -1" rpy="0 0 0" />
+     <joint name="odom_joint" type="fixed">
+        <origin xyz="0 0 0" rpy="0 0 0" />
         <parent link="world" />
         <child link="base_link" />

File: src/dossarm_description/urdf/links_joints.xacro (robot description, xacro)
@@ -16,8 +16,8 @@
       <type>transmission_interface/SimpleTransmission</type>
       <joint name="${name}">
-        <hardwareInterface>hardware_interface/EffortJointInterface</hardwareInterface>
+        <hardwareInterface>hardware_interface/PositionJointInterface</hardwareInterface>
       </joint>
       <actuator name="motor_${name}">
-        <hardwareInterface>hardware_interface/EffortJointInterface</hardwareInterface>
+        <hardwareInterface>hardware_interface/PositionJointInterface</hardwareInterface>
         <mechanicalReduction>1</mechanicalReduction>
       </actuator>
